Commit message: Updated comment in figure_eight.launch, debugged arm_basics.launch and added rviz file for 2-dof arm

File: urdf/twoarm.urdf.xacro (robot description, xacro)
@@ -1,83 +1,86 @@
-<!-- Get properties from arm.yaml configuration -->
-<xacro:property name="arm_yaml_file" value="$(find homework2)/config/arm.yaml"/>
-<xacro:property name="arm_props" value="${load_yaml(yaml_file)}"/>
-<!-- Properties from arm.yaml -->
-<xacro:property name="L1" value="arm_props['L1']"/>
-<xacro:property name="L2" value="arm_props['L2']"/>
-<xacro:property name="R1" value="arm_props['R1']"/>
-<xacro:property name="R2" value="arm_props['R2']"/>
-<xacro:property name="pi" value="3.14159"/>
-<!-- Links -->
-<link name="base_link"/>
-<link name="link_1">
-    <visual>
-        <origin xyz="${L1}/2 0 0" rpy="${pi}/2 0 ${pi}/2"/>
-        <geometry>
-            <cylinder length="${L1}" radius="${R1}"/>
-        </geometry>
-        <material name="blue">
-            <color rgba="0 0 .8 1"/>
-        </material>
-    </visual>
-    <collision>
-        <origin xyz="${L1}/2 0 0" rpy="${pi}/2 0 ${pi}/2"/>
-        <geometry>
-            <cylinder length="${L1}" radius="${R1}"/>
-        </geometry>
-    </collision>
-    <inertial>
-        <origin xyz="${L1}/2 0 0" rpy="${pi}/2 0 ${pi}/2"/>
-        <mass value="1"/>
-        <inertia ixx="${(1.0/12.0)*(3*R1 + L1**2)}"
-                 ixy="0"
-                 ixz="0"
-                 iyy="${(1.0/12.0)*(3*R1 + L1**2)}"
-                 iyz="0"
-                 izz="${0.5*R1**2}"/>
-    </inertial>
-</link>
-<link name="link_2">
-    <visual>
-        <origin xyz="${L2}/2 0 0" rpy="${pi}/2 0 ${pi}/2"/>
-        <geometry>
-            <cylinder length="${L2}" radius="${R2}"/>
-        </geometry>
-        <material name="red">
-            <color rgba=".8 0 0 1"/>
-        </material>
-    </visual>
-    <collision>
-        <origin xyz="${L2}/2 0 0" rpy="${pi}/2 0 ${pi}/2"/>
-        <geometry>
-            <cylinder length="${L2}" radius="${R2}"/>
-        </geometry>
-    </collision>
-    <inertial>
-        <origin xyz="${L2}/2 0 0" rpy="${pi}/2 0 ${pi}/2"/>
-        <mass value="1"/>
-        <inertia ixx="${(1.0/12.0)*(3*R2 + L2**2)}"
-                 ixy="0"
-                 ixz="0"
-                 iyy="${(1.0/12.0)*(3*R2 + L2**2)}"
-                 iyz="0"
-                 izz="${0.5*R2**2}"/>
-    </inertial>
-</link>
-<link name="link_3"/>
-<!-- Joints -->
-<joint name="joint_1" type="continuous">
-    <parent link="base_link"/>
-    <child link="link_1"/>
-    <origin xyz="0 0 0"/>
-    <axis xyz="0 0 1"/>
-</joint>
-<joint name="joint_2" type="continuous">
-    <parent link="link_1">
-    <child link="link_2"/>
-    <origin xyz="${L1} 0 0"/>
-    <axis xyz="0 0 1"/>
-</joint name="end_effector" type="fixed">
-    <parent link="link_2">
-    <child link="link_3">
-    <origin xyz="${L2} 0 0"/>
-</joint>
+<?xml version="1.0"?>
+<robot name="arm" xmlns:xacro="https://www.ros.org/wiki/xacro">
+    <!-- Get properties from arm.yaml configuration -->
+    <xacro:property name="arm_yaml_file" value="$(find homework2)/config/arm.yaml"/>
+    <xacro:property name="arm_props" value="${load_yaml(arm_yaml_file)}"/>
+    <!-- Properties from arm.yaml -->
+    <xacro:property name="L1" value="${arm_props['L1']}"/>
+    <xacro:property name="L2" value="${arm_props['L2']}"/>
+    <xacro:property name="R1" value="${arm_props['R1']}"/>
+    <xacro:property name="R2" value="${arm_props['R2']}"/>
+    <!-- Links -->
+    <link name="base_link"/>
+    <link name="link_1">
+        <visual>
+            <origin xyz="${L1/2} 0 0" rpy="${pi/2} 0 ${pi/2}"/>
+            <geometry>
+                <cylinder length="${L1}" radius="${R1}"/>
+            </geometry>
+            <material name="blue">
+                <color rgba="0 0 .8 1"/>
+            </material>
+        </visual>
+        <collision>
+            <origin xyz="${L1/2} 0 0" rpy="${pi/2} 0 ${pi/2}"/>
+            <geometry>
+                <cylinder length="${L1}" radius="${R1}"/>
+            </geometry>
+        </collision>
+        <inertial>
+            <origin xyz="${L1/2} 0 0" rpy="${pi/2} 0 ${pi/2}"/>
+            <mass value="1"/>
+            <inertia ixx="${(1.0/12.0)*(3*R1 + L1**2)}"
+                    ixy="0"
+                    ixz="0"
+                    iyy="${(1.0/12.0)*(3*R1 + L1**2)}"
+                    iyz="0"
+                    izz="${0.5*R1**2}"/>
+        </inertial>
+    </link>
+    <link name="link_2">
+        <visual>
+            <origin xyz="${L2/2} 0 0" rpy="${pi/2} 0 ${pi/2}"/>
+            <geometry>
+                <cylinder length="${L2}" radius="${R2}"/>
+            </geometry>
+            <material name="red">
+                <color rgba=".8 0 0 1"/>
+            </material>
+        </visual>
+        <collision>
+            <origin xyz="${L2/2} 0 0" rpy="${pi/2} 0 ${pi/2}"/>
+            <geometry>
+                <cylinder length="${L2}" radius="${R2}"/>
+            </geometry>
+        </collision>
+        <inertial>
+            <origin xyz="${L2/2} 0 0" rpy="${pi/2} 0 ${pi/2}"/>
+            <mass value="1"/>
+            <inertia ixx="${(1.0/12.0)*(3*R2 + L2**2)}"
+                    ixy="0"
+                    ixz="0"
+                    iyy="${(1.0/12.0)*(3*R2 + L2**2)}"
+                    iyz="0"
+                    izz="${0.5*R2**2}"/>
+        </inertial>
+    </link>
+    <link name="link_3"/>
+    <!-- Joints -->
+    <joint name="joint_1" type="continuous">
+        <parent link="base_link"/>
+        <child link="link_1"/>
+        <origin xyz="0 0 0"/>
+        <axis xyz="0 0 1"/>
+    </joint>
+    <joint name="joint_2" type="continuous">
+        <parent link="link_1"/>
+        <child link="link_2"/>
+        <origin xyz="${L1} 0 0"/>
+        <axis xyz="0 0 1"/>
+    </joint>
+    <joint name="end_effector" type="fixed">
+        <parent link="link_2"/>
+        <child link="link_3"/>
+        <origin xyz="${L2} 0 0"/>
+    </joint>
+</robot>

Commit message: Added arm_traj node to publish trajectory of robot, updated twoarm.urdf.xacro to support namespace encapsulation, applied namespace encapsulation to arm.yaml

File: urdf/twoarm.urdf.xacro (robot description, xacro)
@@ -5,8 +5,10 @@
     <xacro:property name="arm_props" value="${load_yaml(arm_yaml_file)}"/>
     <!-- Properties from arm.yaml -->
-    <xacro:property name="L1" value="${arm_props['L1']}"/>
-    <xacro:property name="L2" value="${arm_props['L2']}"/>
-    <xacro:property name="R1" value="${arm_props['R1']}"/>
-    <xacro:property name="R2" value="${arm_props['R2']}"/>
+    <xacro:property name="homework2_ns" value="${arm_props['homework2']}"/>
+    <xacro:property name="twoarm_ns" value="${homework2_ns['twoarm']}"/>
+    <xacro:property name="L1" value="${twoarm_ns['L1']}"/>
+    <xacro:property name="L2" value="${twoarm_ns['L2']}"/>
+    <xacro:property name="R1" value="${twoarm_ns['R1']}"/>
+    <xacro:property name="R2" value="${twoarm_ns['R2']}"/>
     <!-- Links -->
     <link name="base_link"/>

Commit message: Removed python extension on arm_marker, debugged arm marker to allow marker to show on rviz, updated twoarm.rviz and twoarm.urdf.xacro for tf debugging, added arm_marker to CMakeLists

File: urdf/twoarm.urdf.xacro (robot description, xacro)
@@ -12,5 +12,5 @@
     <xacro:property name="R2" value="${twoarm_ns['R2']}"/>
     <!-- Links -->
-    <link name="base_link"/>
+    <link name="base"/>
     <link name="link_1">
         <visual>
@@ -70,5 +70,5 @@
     <!-- Joints -->
     <joint name="joint_1" type="continuous">
-        <parent link="base_link"/>
+        <parent link="base"/>
         <child link="link_1"/>
         <origin xyz="0 0 0"/>
